Commit message: bot and walls spawing without falling

File: person_follower_sim/urdf/mr_robot.xacro (robot description, xacro)
@@ -3,9 +3,17 @@
 <xacro:include filename="$(find person_follower_sim)/urdf/materials.xacro" />
 <xacro:include filename="$(find person_follower_sim)/urdf/mr_robot.trans" />
-<xacro:include filename="$(find person_follower_sim)/gazebo/mr_robot.gazebo" />
-<xacro:include filename="$(find person_follower_sim)/gazebo/mr_robot_plugins.gazebo" />
+<xacro:include filename="$(find person_follower_sim)/urdf/mr_robot.gazebo" />
+<!-- <xacro:include filename="$(find person_follower_sim)/gazebo/mr_robot_plugins.gazebo" /> -->
 <xacro:arg      name="kinect_enabled"             default="true" />
 <xacro:arg      name="lidar_enabled"              default="true" />
 <xacro:arg      name="camera_enabled"             default="true" />
+<link name="imu_link">
+  <visual>
+      <origin xyz="0 0 0" rpy="0 0 0"/>
+    <geometry>
+        <box size="0.02 0.015 0.008"/>
+      </geometry>
+    </visual>
+</link>
 <link name="base_link" gravity="0 0 -9.8">
   <inertial>
@@ -48,4 +56,10 @@
   </collision>
 </link>
+<joint name="imu_joint" type="fixed">
+  <origin xyz="0 0 0.18" rpy="0 0 0"/>
+  <parent link="base_link"/>
+  <child link="imu_link"/>
+  <axis xyz="0 0 0" />
+</joint>
 <link name="l_tyre_1">
   <inertial>
@@ -68,5 +82,4 @@
   </collision>
 </link>
-<xacro:if value="$(arg lidar_enabled)">
 <link name="lidar_1">
   <inertial>
@@ -94,5 +107,4 @@
   <child link="lidar_1"/>
 </joint>
-</xacro:if>
 <xacro:if value="$(arg kinect_enabled)">
 	<link name="kinect_camera">
@@ -106,5 +118,5 @@
 			<origin xyz="0 0 0" rpy="0 0 0" />
 		<geometry>
-		<mesh filename="file://$(find person_follower_sim)/meshes/kinect/d415.dae"/>
+		<mesh filename="package://$(find person_follower_sim)/meshes/kinect/d415.dae"/>
 		</geometry>
 		<material name="black"/>
@@ -121,5 +133,4 @@
 	</joint>
 </xacro:if>
-<xacro:if value="$(arg camera_enabled)">
   <link name="camera_link">
     <collision>
@@ -147,5 +158,4 @@
    <child link="camera_link"/>
   </joint>
-</xacro:if>
 <joint name="right_motor_joint" type="continuous">
   <origin rpy="0 0 0" xyz="-0.003445 -0.10058 0.052283"/>

Commit message: walking_actor

File: person_follower_sim/urdf/mr_robot.xacro (robot description, xacro)
@@ -118,5 +118,5 @@
 			<origin xyz="0 0 0" rpy="0 0 0" />
 		<geometry>
-		<mesh filename="package://$(find person_follower_sim)/meshes/kinect/d415.dae"/>
+		<mesh filename="file://$(find person_follower_sim)/meshes/kinect/d415.dae"/>
 		</geometry>
 		<material name="black"/>

Commit message: camera-image and differential drive

File: person_follower_sim/urdf/mr_robot.xacro (robot description, xacro)
@@ -1,4 +1,4 @@
 <?xml version="1.0" ?>
-<robot name="mr_robot" xmlns:xacro="http://www.ros.org/wiki/xacro">
+<robot name="mr_robot" xmlns:xacro="http://www.ros.org/wiki/xacro" xmlns:gz="http://gazebosim.org/schema">
 <xacro:include filename="$(find person_follower_sim)/urdf/materials.xacro" />
 <xacro:include filename="$(find person_follower_sim)/urdf/mr_robot.trans" />
@@ -118,5 +118,5 @@
 			<origin xyz="0 0 0" rpy="0 0 0" />
 		<geometry>
-		<mesh filename="file://$(find person_follower_sim)/meshes/kinect/d415.dae"/>
+		<mesh filename="file://$(find person_follower_sim)/meshes/kinect/../realsense_texture.png"/>
 		</geometry>
 		<material name="black"/>
